Commit message: Mejorado

File: robot_grua/urdf/robot_grua_rviz.urdf (robot description, URDF)
Before this commit: robot grua, 7 links, 6 joints
Links:
- link link0: geometry visual mesh filename=package://robot_grua/urdf/stl_parts/base.stl scale=0.01 0.01 0.01
- link link1: geometry visual mesh filename=package://robot_grua/urdf/stl_parts/link1.stl scale=0.01 0.01 0.01
- link link2: geometry visual mesh filename=package://robot_grua/urdf/stl_parts/link2.stl scale=0.01 0.01 0.01
- link link3: geometry visual mesh filename=package://robot_grua/urdf/stl_parts/link3.stl scale=0.01 0.01 0.01
- link link4: geometry visual mesh filename=package://robot_grua/urdf/stl_parts/link4.stl scale=0.01 0.01 0.01
- link link5: geometry visual mesh filename=package://robot_grua/urdf/stl_parts/link5.stl scale=0.01 0.01 0.01
- link link6: geometry visual mesh filename=package://robot_grua/urdf/stl_parts/link6.stl scale=0.01 0.01 0.01
